File: Hardware/SparkFun_QRE1113_Line_Sensor_Breakout_Digital.brd (EAGLE design)
At the start: 7.6 x 14 mm, 7 parts, among them U1 QRE1113

Commit message: added board fiducials
Parts:
- added FID1, FID2: FIDUCIALUFIDUCIAL, SparkFun-Aesthetics:MICRO-FIDUCIAL
